Commit message: 3333

File: widowx-project/widowx_arm/widowx_arm_description/robots/widowx_arm.urdf.xacro (robot description, xacro)
@@ -2,13 +2,7 @@
 <robot name="widowx_arm" xmlns:xacro="http://ros.org/wiki/xacro">
 	<xacro:include filename="$(find widowx_arm_description)/urdf/widowx.urdf.xacro"/>
-	<link name="base_footprint">
-		<visual>
-			<origin xyz="0 0 0" rpy="0 0 0"/>
-			<geometry>
-				<box size="0.001 0.001 0.001" />
-			</geometry>
-		</visual>
+	<link name="world">
 	</link>
-	<xacro:widowx_arm parent="base_footprint" prefix="">
+	<xacro:widowx_arm parent="world" prefix="">
 		<origin xyz="0.0 0.0 0.0" rpy="0.0 0.0 0.0"/>
 	</xacro:widowx_arm>

Commit message: 5545345

File: widowx-project/widowx_arm/widowx_arm_description/robots/widowx_arm.urdf.xacro (robot description, xacro)
@@ -2,7 +2,13 @@
 <robot name="widowx_arm" xmlns:xacro="http://ros.org/wiki/xacro">
 	<xacro:include filename="$(find widowx_arm_description)/urdf/widowx.urdf.xacro"/>
-	<link name="world">
+	<link name="base_footprint">
+		<visual>
+			<origin xyz="0 0 0" rpy="0 0 0"/>
+			<geometry>
+				<box size="0.001 0.001 0.001" />
+			</geometry>
+		</visual>
 	</link>
-	<xacro:widowx_arm parent="world" prefix="">
+	<xacro:widowx_arm parent="base_footprint" prefix="">
 		<origin xyz="0.0 0.0 0.0" rpy="0.0 0.0 0.0"/>
 	</xacro:widowx_arm>
